File: Esp32_IO_1-wire.kicad_pcb (KiCad board)
At the start: 2 copper layers, 50 x 100 mm, 29 parts, among them J1 IO-pins, J2 1-Wire, J3 Vin, J4 I2C, J5 GPIO -pins, J6 RX/TX, U1 DS2484R, U2 PCF8574AT, U3 ESP32_S3_supermini

Commit message: Signed-off-by: regamp <patbence1999@gmail.com>
Routing:
- net +3.3V: track 43.6 -> 46.5 mm, vias 2 -> 4
- net Net-(U3-TX): track 43.8 -> 45.4 mm

Commit message: I2C Bus with 1,27mm pinheader
Parts:
- removed A0, A1, A2: SolderJumper_3_Open, Jumper:SolderJumper-3_P1.3mm_Open_RoundedPad1.0x1.5mm_NumberLabels
- added J7: I2C bus, Connector_PinHeader_1.27mm:PinHeader_1x03_P1.27mm_Horizontal, F.Cu at (122.8, 135.9)
- added JP4: SolderJumper_3_Open, Jumper:SolderJumper-3_P1.3mm_Open_RoundedPad1.0x1.5mm_NumberLabels, B.Cu at (121.9, 130.5)
- added JP5: SolderJumper_3_Open, Jumper:SolderJumper-3_P1.3mm_Open_RoundedPad1.0x1.5mm_NumberLabels, B.Cu at (121.8, 127.4)
- added JP6: SolderJumper_3_Open, Jumper:SolderJumper-3_P1.3mm_Open_RoundedPad1.0x1.5mm_NumberLabels, B.Cu at (121.8, 124.6)
Routing:
- net /SCL: track 48.7 -> 70.7 mm
- net /SDA: track 50.6 -> 70.2 mm
Other:
- board text added: "I2C Bus+GND"

Commit message: Logo
Parts:
- added REF**: KiCad-Logo2_5mm_SilkScreen, Symbol:KiCad-Logo2_5mm_SilkScreen, B.Cu at (158.4, 135.7)
Other:
- board text added: "100mm"
- board text added: "60mm"
- board text added: "Designed by Bence"
- board text added: "https://github.com/regamp/ESP32-S3-1-WIRE"
- board text removed: "60 mm"

Commit message: I2C routing fix
Parts:
- moved TP3 4.51 mm to (127.5, 131.8)
Routing:
- net /SCL: track 70.7 -> 65.7 mm, vias 1 -> 0
- net /SDA: track 70.2 -> 72.6 mm, vias 1 -> 0
- net +3.3V: track 46.5 -> 48.6 mm, vias 4 -> 6
- net GND: track 12.5 -> 13.2 mm
- net /1-Wire: track 16.9 -> 17.0 mm, vias 0 -> 1

Commit message: via
Parts:
- removed TP3: 1-W, TestPoint:TestPoint_Pad_D1.0mm
- moved R4 1.26 mm to (127.0, 134.6)
Routing:
- net +3.3V: track 48.6 -> 48.1 mm
Other:
- board text removed: "https://github.com/regamp/ESP32-S3-1-WIRE"
Changed lines of the file:
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@@
 		(tags "capacitor handsolder")
 		(property "Reference" "C3"
-			(at -3.0125 -0.075 0)
+			(at -3.7875 0 0)
 			(layer "F.SilkS")
 			(effects
@@
 		)
 	)
-	(footprint "TestPoint:TestPoint_Pad_D1.0mm"
-		(layer "F.Cu")
-		(at 127.5 131.775)
-		(descr "SMD pad as test Point, diameter 1.0mm")
-		(tags "test point SMD pad")
-		(property "Reference" "TP3"
-			(at 0 -1.448 0)
-			(layer "F.SilkS")
-			(effects
-				(font
-					(size 1 1)
-					(thickness 0.15)
-				)
-			)
-		)
-		(property "Value" "1-W"
-			(at 0.2 1.125 0)
-			(layer "F.SilkS")
-			(effects
-				(font
-					(size 1 1)
-					(thickness 0.15)
-				)
-			)
-		)
-		(property "Datasheet" ""
-			(at 0 0 0)
-			(unlocked yes)
-			(layer "F.Fab")
-			(hide yes)
-			(effects
-				(font
-					(size 1.27 1.27)
-					(thickness 0.15)
-				)
-			)
-		)
-		(property "Description" "test point"
-			(at 0 0 0)
-			(unlocked yes)
-			(layer "F.Fab")
-			(hide yes)
-			(effects
-				(font
-					(size 1.27 1.27)
-					(thickness 0.15)
-				)
-			)
-		)
-		(property ki_fp_filters "Pin* Test*")
-		(sheetname "/")
-		(sheetfile "Esp32_IO_1-wire.kicad_sch")
-		(units
-			(unit
-				(name "A")
-				(pins "1")
-			)
-		)
-		(duplicate_pad_numbers_are_jumpers no)
-		(fp_circle
-			(center 0 0)
-			(end 0 0.7)
-			(stroke
-				(width 0.12)
-				(type solid)
-			)
-			(fill no)
-			(layer "F.SilkS")
-		)
-		(fp_circle
-			(center 0 0)
-			(end 1 0)
-			(stroke
-				(width 0.05)
-				(type solid)
-			)
-			(fill no)
-			(layer "F.CrtYd")
-		)
-		(fp_text user "${REFERENCE}"
-			(at 0 -1.45 0)
-			(layer "F.Fab")
-			(effects
-				(font
-					(size 1 1)
-					(thickness 0.15)
-				)
-			)
-		)
-		(pad "1" smd circle
-			(at 0 0)
-			(size 1 1)
-			(layers "F.Cu" "F.Mask")
-			(net "/1-Wire")
-			(pinfunction "1_1")
-			(pintype "passive")
-		)
-		(embedded_fonts no)
-	)
 	(footprint "Resistor_SMD:R_0805_2012Metric_Pad1.20x1.40mm_HandSolder"
 		(layer "F.Cu")
@@
 	(footprint "Resistor_SMD:R_0805_2012Metric_Pad1.20x1.40mm_HandSolder"
 		(layer "F.Cu")
-		(at 125.775 134.775 90)
+		(at 127.025 134.625 90)
 		(descr "Resistor SMD 0805 (2012 Metric), square (rectangular) end terminal, IPC-7351 nominal with elongated pad for handsoldering. (Body size source: IPC-SM-782 page 72, https://www.pcb-3d.com/wordpress/wp-content/uploads/ipc-sm-782a_amendment_1_and_2.pdf)")
 		(tags "resistor handsolder")
@@
 		(tags "capacitor handsolder")
 		(property "Reference" "C2"
-			(at -3.3875 0.01 0)
+			(at -3.7875 -0.025 0)
 			(layer "F.SilkS")
 			(effects
@@
 	(gr_line
 		(start 122 123.05)
-		(end 124.725 123.05)
+		(end 125.4625 123.05)
 		(stroke
 			(width 0.1)
@@
 	)
 	(gr_line
-		(start 124.7 136.85)
-		(end 124.725 123.05)
+		(start 125.4375 136.85)
+		(end 125.4625 123.05)
 		(stroke
 			(width 0.1)
@@
 	)
 	(gr_line
-		(start 124.7 136.85)
+		(start 125.4375 136.85)
 		(end 128.25 136.85)
 		(stroke
@@
 		(layer "Margin")
 	)
+	(gr_text "GND"
+		(at 123.875 133.6 0)
+		(layer "F.SilkS")
+		(effects
+			(font
+				(size 0.5 0.5)
+				(thickness 0.1)
+				(bold yes)
+			)
+			(justify left bottom)
+		)
+	)
+	(gr_text "SCL"
+		(at 123.875 135.025 0)
+		(layer "F.SilkS")
+		(effects
+			(font
+				(size 0.5 0.5)
+				(thickness 0.1)
+				(bold yes)
+			)
+			(justify left bottom)
+		)
+	)
+	(gr_text "SDA"
+		(at 123.9 136.4 0)
+		(layer "F.SilkS")
+		(effects
+			(font
+				(size 0.5 0.5)
+				(thickness 0.1)
+				(bold yes)
+			)
+			(justify left bottom)
+		)
+	)
 	(gr_text "I2C Bus+GND"
 		(at 119.525 132.3 90)
@@
 		)
 	)
-	(gr_text "https://github.com/regamp/ESP32-S3-1-WIRE"
-		(at 160.2 112.275 0)
-		(layer "B.SilkS")
-		(effects
-			(font
-				(size 1 1)
-				(thickness 0.1)
-			)
-			(justify left bottom mirror)
-		)
-	)
 	(gr_text "Designed by Bence"
 		(at 164.95 131.575 0)
@@
 	)
 	(segment
-		(start 125.775 135.875)
-		(end 129.575 139.675)
+		(start 127.025 135.625)
+		(end 127.025 136.45)
 		(width 0.5)
 		(layer "F.Cu")
@@
 	)
 	(segment
-		(start 138.5 118.725)
-		(end 138.5 117.425)
-		(width 2)
-		(layer "F.Cu")
-		(net "+3.3V")
-	)
-	(segment
-		(start 129.575 139.675)
-		(end 129.575 139.7)
+		(start 127.025 136.45)
+		(end 129.925 139.35)
 		(width 0.5)
 		(layer "F.Cu")
@@
 	)
 	(segment
-		(start 125.775 135.775)
-		(end 125.775 135.875)
-		(width 0.5)
+		(start 138.5 118.725)
+		(end 138.5 117.425)
+		(width 2)
 		(layer "F.Cu")
 		(net "+3.3V")
@@
 	)
 	(via
-		(at 129.575 139.7)
+		(at 129.925 139.35)
 		(size 0.6)
 		(drill 0.3)
@@
 	)
 	(segment
-		(start 136.5 116.325)
-		(end 136.85 116.675)
-		(width 0.2)
-		(layer "B.Cu")
-		(net "+3.3V")
-	)
-	(segment
-		(start 136.85 116.675)
-		(end 136.85 117.875)
-		(width 0.2)
+		(start 128 141.275)
+		(end 128 144.5)
+		(width 1)
 		(layer "B.Cu")
 		(net "+3.3V")
 	)
 	(segment
-		(start 128 144.5)
-		(end 128 141.275)
+		(start 129.925 139.35)
+		(end 135.875 139.35)
 		(width 1)
 		(layer "B.Cu")
@@
 	)
 	(segment
-		(start 128 141.275)
-		(end 129.575 139.7)
+		(start 129.925 139.35)
+		(end 128 141.275)
 		(width 1)
 		(layer "B.Cu")
@@
 	)
 	(segment
-		(start 137.85 136.05)
+		(start 135.875 139.35)
 		(end 137.85 137.375)
 		(width 1)
@@
 	)
 	(segment
-		(start 135.875 139.35)
-		(end 137.85 137.375)
-		(width 1)
+		(start 136.5 116.325)
+		(end 136.85 116.675)
+		(width 0.2)
 		(layer "B.Cu")
 		(net "+3.3V")
 	)
 	(segment
-		(start 129.575 139.7)
-		(end 129.925 139.35)
-		(width 1)
+		(start 136.85 116.675)
+		(end 136.85 117.875)
+		(width 0.2)
 		(layer "B.Cu")
 		(net "+3.3V")
 	)
 	(segment
-		(start 129.925 139.35)
-		(end 135.875 139.35)
+		(start 137.85 136.05)
+		(end 137.85 137.375)
 		(width 1)
 		(layer "B.Cu")
@@
 	)
 	(segment
+		(start 127.025 133.625)
+		(end 127.025 133.075)
+		(width 0.25)
+		(layer "F.Cu")
+		(net "Net-(JP4-A)")
+	)
+	(segment
 		(start 125.775 127.1)
 		(end 125.775 124.65)
@@
 	)
 	(segment
-		(start 125.775 131.825)
-		(end 125.775 127.1)
+		(start 127.025 133.075)
+		(end 125.775 131.825)
 		(width 0.5)
 		(layer "F.Cu")
@@
 	)
 	(segment
-		(start 125.775 133.775)
-		(end 125.775 131.825)
+		(start 125.775 131.825)
+		(end 125.775 127.1)
 		(width 0.5)
 		(layer "F.Cu")
@@
 		(layer "F.Cu")
 		(hatch edge 0.5)
-		(connect_pads yes
+		(connect_pads
 			(clearance 0.5)
 		)
@@
 		(hatch edge 0.5)
 		(priority 1)
-		(connect_pads yes
+		(connect_pads
 			(clearance 0.5)
 		)
@@
 		(priority 2)
 		(connect_pads
-			(clearance 0.5)
+			(clearance 0.4)
 		)
 		(min_thickness 0.25)

Commit message: pacman
Parts:
- added G***: LOGO, Library:pacman, F.Cu at (140.4, 65.1)
